File: I2CRJ45X24.brd (EAGLE design)
At the start: 275 x 50 mm, 123 parts, among them IC1 MCP23017SO, IC2 MCP23017SO, IC3 MCP23017SO, IC4 MCP23017SO, IC5 MCP23017SO, IC6 MCP23017SO, J1 RJ45-X8, J2 RJ45-X8, J3 RJ45-X8, J5 M06-PIN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

Commit message: Update I2CRJ45X24.brd
Routing:
- net SDA: track 126.9 -> 224.6 mm, vias 4 -> 6
- net SCL: track 137.0 -> 226.3 mm, vias 5 -> 6
- net VCC: track 231.3 -> 299.2 mm, vias 1 -> 3
- net !INT: track 344.9 -> 381.1 mm
